File: schematics/Program_Counter.kicad_sch (KiCad schematic)
At the start: 46 parts, among them U1 74LS161, U2 74LS161, U3 74LS245, U4 74LS161, U5 74LS161, U6 74LS245, U7 74LS245

Commit message: Updated schematics and README
Connections:
- net CLK: no longer U1.1 (~{MR}), U1.7 (CEP), U1.9 (~{PE}), U2.1 (~{MR}), U2.10 (CET), U2.7 (CEP), U2.9 (~{PE}), U4.1 (~{MR}), U4.15 (TC), U4.7 (CEP), U4.9 (~{PE}), U5.1 (~{MR}), U5.10 (CET), U5.7 (CEP), U5.9 (~{PE})
- new net: U2.10 (CET), U4.15 (TC)
- new net PC_E: U1.7 (CEP), U2.7 (CEP), U4.7 (CEP), U5.10 (CET), U5.7 (CEP)
- new net |PC_IN_16: U1.9 (~{PE}), U2.9 (~{PE}), U4.9 (~{PE}), U5.9 (~{PE})
- new net |RST: U1.1 (~{MR}), U2.1 (~{MR}), U4.1 (~{MR}), U5.1 (~{MR})
Changed lines of the file:
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@@
-	)
-	(junction
-		(at 176.53 80.01)
-		(diameter 0)
-		(color 0 0 0 0)
-	)
-	(junction
-		(at 184.15 85.09)
-		(diameter 0)
-		(color 0 0 0 0)
 	)
 	(junction
@@
 	)
 	(junction
-		(at 181.61 82.55)
-		(diameter 0)
-		(color 0 0 0 0)
-	)
-	(junction
 		(at 53.34 140.97)
 		(diameter 0)
@@
 	)
 	(junction
-		(at 229.87 85.09)
-		(diameter 0)
-		(color 0 0 0 0)
-	)
-	(junction
 		(at 55.88 121.92)
 		(diameter 0)
@@
 	(wire
 		(pts
-			(xy 181.61 80.01) (xy 181.61 82.55)
-		)
-		(stroke
-			(width 0)
-			(type default)
-		)
-	)
-	(wire
-		(pts
 			(xy 58.42 120.65) (xy 135.89 120.65)
 		)
@@
 	(wire
 		(pts
-			(xy 184.15 85.09) (xy 184.15 86.36)
-		)
-		(stroke
-			(width 0)
-			(type default)
-		)
-	)
-	(wire
-		(pts
-			(xy 189.23 85.09) (xy 184.15 85.09)
-		)
-		(stroke
-			(width 0)
-			(type default)
-		)
-	)
-	(wire
-		(pts
-			(xy 176.53 80.01) (xy 176.53 86.36)
+			(xy 184.15 83.82) (xy 184.15 86.36)
+		)
+		(stroke
+			(width 0)
+			(type default)
+		)
+	)
+	(wire
+		(pts
+			(xy 146.05 85.09) (xy 189.23 85.09)
+		)
+		(stroke
+			(width 0)
+			(type default)
+		)
+	)
+	(wire
+		(pts
+			(xy 176.53 77.47) (xy 176.53 86.36)
 		)
 		(stroke
@@
 	(wire
 		(pts
-			(xy 189.23 85.09) (xy 229.87 85.09)
+			(xy 189.23 85.09) (xy 232.41 85.09)
 		)
 		(stroke
@@
 	(wire
 		(pts
-			(xy 138.43 80.01) (xy 176.53 80.01)
-		)
-		(stroke
-			(width 0)
-			(type default)
-		)
-	)
-	(wire
-		(pts
 			(xy 66.04 72.39) (xy 153.67 72.39)
 		)
@@
 	(wire
 		(pts
-			(xy 181.61 80.01) (xy 176.53 80.01)
+			(xy 138.43 80.01) (xy 181.61 80.01)
 		)
 		(stroke
@@
 	(wire
 		(pts
-			(xy 146.05 85.09) (xy 184.15 85.09)
-		)
-		(stroke
-			(width 0)
-			(type default)
-		)
-	)
-	(wire
-		(pts
 			(xy 262.89 77.47) (xy 262.89 86.36)
 		)
@@
 	(wire
 		(pts
-			(xy 143.51 82.55) (xy 181.61 82.55)
-		)
-		(stroke
-			(width 0)
-			(type default)
-		)
-	)
-	(wire
-		(pts
 			(xy 147.32 124.46) (xy 147.32 137.16)
 		)
@@
 	(wire
 		(pts
-			(xy 176.53 77.47) (xy 176.53 80.01)
-		)
-		(stroke
-			(width 0)
-			(type default)
-		)
-	)
-	(wire
-		(pts
-			(xy 229.87 85.09) (xy 232.41 85.09)
-		)
-		(stroke
-			(width 0)
-			(type default)
-		)
-	)
-	(wire
-		(pts
 			(xy 110.49 54.61) (xy 110.49 86.36)
 		)
@@
 	(wire
 		(pts
-			(xy 229.87 82.55) (xy 229.87 85.09)
+			(xy 229.87 82.55) (xy 229.87 86.36)
 		)
 		(stroke
@@
 	(wire
 		(pts
-			(xy 181.61 82.55) (xy 181.61 86.36)
+			(xy 181.61 80.01) (xy 181.61 86.36)
 		)
 		(stroke
@@
 	(wire
 		(pts
-			(xy 184.15 83.82) (xy 184.15 85.09)
-		)
-		(stroke
-			(width 0)
-			(type default)
-		)
-	)
-	(wire
-		(pts
 			(xy 95.25 39.37) (xy 285.75 39.37)
 		)
@@
 	(wire
 		(pts
-			(xy 186.69 82.55) (xy 181.61 82.55)
+			(xy 143.51 82.55) (xy 186.69 82.55)
 		)
 		(stroke
@@
 		)
 		(stroke
-			(width 0)
-			(type default)
-		)
-	)
-	(wire
-		(pts
-			(xy 229.87 85.09) (xy 229.87 86.36)
-		)
-		(stroke
